File: Hardware/pcb.brd (EAGLE design)
At the start: 170.2 x 111.2 mm, 103 parts, among them IC1 BD5229G-TR, IC4 XC6220A331MR-G, J1 FH34SRJ-24S-0.5SH_99_, J2 SAMACSYS_PARTS_USB4110-GF-A, J3 QWIIC_RIGHT_ANGLE, J4 112A-TAAR-R03_ATTEND, Q1 20V/4.2A/52mΩ/1.4W, Q2 20V/4.2A/52mΩ/1.4W, Q3 SI1308EDL-T1-GE3, U1 W25Q512JVEIQ, U2 ESP32-C6-WROOM-1-N8, U3 DS3231SN#, U4 MAX17048G+T10

Commit message: last issues
Parts:
- CHG_LED: value (none) -> LED
- SJ1: value (none) -> SJ
- renumbered 3V3 to TP16, EPD_3V3 to TP17, EPD_3V3_C to TP13, EPD_BUSY to TP9, EPD_CS to TP10, EPD_DC to TP11, EPD_RST to TP12, GND to TP4, GND_2 to TP5, INT_RTC to TP15, MISO to TP6, MOSI to TP7, RX to TP2, SCK to TP8, TX to TP1, VBAT to TP3, VBUS to TP14
Routing:
- net RESE: track 25.0 -> 51.4 mm, vias 2 -> 0
- net SCK: track 178.8 -> 189.8 mm
- net EPD_BUSY: track 117.7 -> 109.0 mm, vias 4 -> 3
- net MISO: track 140.5 -> 148.3 mm, vias 5 -> 4
- net MOSI: track 160.8 -> 167.7 mm, vias 6 -> 5
- net GDR: track 26.7 -> 31.2 mm
- net 3V3: track 396.5 -> 393.6 mm
- net SCL: track 201.9 -> 199.1 mm, vias 6 -> 7
- net EPD_RST: track 116.1 -> 113.5 mm
- net SDA: track 187.9 -> 185.5 mm
- net PREVGH: track 25.7 -> 27.6 mm
- net FLASH_CS: track 21.7 -> 20.0 mm
- net EPD_CS: track 109.3 -> 107.8 mm
- net EPD_3V3: track 51.4 -> 52.7 mm, vias 3 -> 4
- net INT_RTC: track 108.2 -> 109.2 mm
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Other:
- board text added: "3V3"
- board text added: "EPD_3V3"
- board text added: "EPD_3V3_C"
- board text added: "EPD_BUSY"
- board text added: "EPD_CS"
- board text added: "EPD_DC"
- board text added: "EPD_RST"
- board text added: "GND"
- board text added: "INT_RTC"
- board text added: "MISO"
- board text added: "MOSI"
- board text added: "RX"
- board text added: "SCK"
- board text added: "TX"
- board text added: "VBAT"
- board text added: "VBUS"
