File: Hardware/schematic.sch (EAGLE design)
At the start: 103 parts, among them IC1 BD5229G-TR, IC4 XC6220A331MR-G, J1 FH34SRJ-24S-0.5SH_99_, J2 SAMACSYS_PARTS_USB4110-GF-A, J3 QWIIC_RIGHT_ANGLE, J4 112A-TAAR-R03_ATTEND, Q1 20V/4.2A/52mΩ/1.4W, Q2 20V/4.2A/52mΩ/1.4W, Q3 SI1308EDL-T1-GE3, U1 W25Q512JVEIQ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

Commit message: last issues
Parts:
- CHG_LED: value (none) -> LED
- SJ1: value (none) -> SJ
- renumbered 3V3 to TP16, EPD_3V3 to TP17, EPD_3V3_C to TP13, EPD_BUSY to TP9, EPD_CS to TP10, EPD_DC to TP11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
